Commit message: update

File: src/urdf_tutorial/urdf/06-flexible.urdf (robot description, URDF)
Before this commit: robot visual, 16 links, 15 joints
Joints:
- removed joint tobox
- joint base_to_right_leg: axis (none) -> 0 0 1; limit (none) -> lower=0.0 upper=0.548 effort=1000.0 velocity=0.5; origin xyz=0 -0.22 0.25 -> xyz=-0.0032186 0 -0.00093742 rpy=1.5708 1.2516 -1.5708; type fixed -> revolute
