Commit message: update

File: src/robot_arm_urdf/urdf/robot_arm_urdf.urdf (robot description, URDF)
Before this commit: robot robot_arm_urdf, 12 links, 11 joints
Joints:
- joint right_gripper1_joint: limit lower=-1.5708 upper=0 effort=1000 velocity=0.5 -> lower=-1.5708 upper=1.5708 effort=1000 velocity=0.5

Commit message: update

File: src/robot_arm_urdf/urdf/robot_arm_urdf.urdf (robot description, URDF)
Before this commit: robot robot_arm_urdf, 12 links, 11 joints
Joints:
- joint fifth_joint: origin xyz=0.031 -0.04815 0.031 rpy=3.1416 6.0177E-09 -1.5708 -> xyz=0.031 -0.04815 0.031 rpy=1.5708 6.0177E-09 -1.5708

Commit message: update

File: src/robot_arm_urdf/urdf/robot_arm_urdf.urdf (robot description, URDF)
Before this commit: robot robot_arm_urdf, 12 links, 11 joints
Joints:
- joint left_gripper1_joint: limit lower=-1.5708 upper=0 effort=1000 velocity=0.5 -> lower=-1.5708 upper=1.5708 effort=1000 velocity=0.5
- joint left_gripper2_joint: limit lower=-1.5708 upper=0 effort=1000 velocity=0.5 -> lower=-1.5708 upper=1.5708 effort=1000 velocity=0.5
- joint left_gripper3_joint: limit lower=-1.5708 upper=0 effort=1000 velocity=0.5 -> lower=-1.5708 upper=1.5708 effort=1000 velocity=0.5
- joint right_gripper2_joint: limit lower=0 upper=1.5708 effort=1000 velocity=0.5 -> lower=-1.5708 upper=1.5708 effort=1000 velocity=0.5
- joint right_gripper3_joint: limit lower=-1.5708 upper=0 effort=1000 velocity=0.5 -> lower=-1.5708 upper=1.5708 effort=1000 velocity=0.5

Commit message: update

File: src/robot_arm_urdf/urdf/robot_arm_urdf.urdf (robot description, URDF)
Before this commit: robot robot_arm_urdf, 12 links, 11 joints
Joints:
- joint fifth_joint: limit lower=-1.5708 upper=1.5708 effort=1000 velocity=0.5 -> lower=-1.5708 upper=1.5708 effort=1000 velocity=5
- joint first_joint: limit lower=-1.5708 upper=1.5708 effort=1000 velocity=0.5 -> lower=-1.5708 upper=1.5708 effort=1000 velocity=5
- joint fourth_joint: limit lower=-1.5708 upper=1.5708 effort=1000 velocity=0.5 -> lower=-1.5708 upper=1.5708 effort=1000 velocity=5
- joint left_gripper1_joint: limit lower=-1.5708 upper=1.5708 effort=1000 velocity=0.5 -> lower=-1.5708 upper=1.5708 effort=1000 velocity=5
- joint left_gripper2_joint: limit lower=-1.5708 upper=1.5708 effort=1000 velocity=0.5 -> lower=-1.5708 upper=1.5708 effort=1000 velocity=5
- joint left_gripper3_joint: limit lower=-1.5708 upper=1.5708 effort=1000 velocity=0.5 -> lower=-1.5708 upper=1.5708 effort=1000 velocity=5
- joint right_gripper1_joint: limit lower=-1.5708 upper=1.5708 effort=1000 velocity=0.5 -> lower=-1.5708 upper=1.5708 effort=1000 velocity=5
- joint right_gripper2_joint: limit lower=-1.5708 upper=1.5708 effort=1000 velocity=0.5 -> lower=-1.5708 upper=1.5708 effort=1000 velocity=5
- joint right_gripper3_joint: limit lower=-1.5708 upper=1.5708 effort=1000 velocity=0.5 -> lower=-1.5708 upper=1.5708 effort=1000 velocity=5
- joint second_joint: limit lower=-1.5708 upper=1.5708 effort=1000 velocity=0.5 -> lower=-1.5708 upper=1.5708 effort=1000 velocity=5
- joint third_joint: limit lower=-1.5708 upper=1.5708 effort=1000 velocity=0.5 -> lower=-1.5708 upper=1.5708 effort=1000 velocity=5
